Commit message: URDF working

File: src/vanderbot/urdf/vanderbot.urdf (robot description, URDF)
Before this commit: robot console.log, 5 links, 4 joints
Links:
- added link world
- link base_link: mass 0.80794 -> None; geometry collision mesh filename=package://vanderbot/meshes/base_link.STL; visual mesh filename=package://vanderbot/meshes/base_link.STL
- link link_1: mass 0.5361 -> None; geometry collision mesh filename=package://vanderbot/meshes/link_1.STL; visual mesh filename=package://vanderbot/meshes/link_1.STL
- link link_2: mass 0.66905 -> None; geometry collision mesh filename=package://vanderbot/meshes/link_2.STL; visual mesh filename=package://vanderbot/meshes/link_2.STL
- link link_3: mass 0.44826 -> None; geometry collision mesh filename=package://vanderbot/meshes/link_3.STL; visual mesh filename=package://vanderbot/meshes/link_3.STL
- link link_4: mass 0.23962 -> None; geometry collision mesh filename=package://vanderbot/meshes/link_4.STL; visual mesh filename=package://vanderbot/meshes/link_4.STL
Joints:
- added joint fix: type fixed, parent world, child base_link, origin xyz=0 0 0 rpy=1.5708 0 0
- joint joint_1: type revolute -> continuous
- joint joint_2: type revolute -> continuous
- joint joint_3: type revolute -> continuous
- joint joint_4: type revolute -> continuous

Commit message: rviz shows changes in arm position but is not properly zeroed

File: src/vanderbot/urdf/vanderbot.urdf (robot description, URDF)
Before this commit: robot vanderbot, 6 links, 5 joints
Joints:
- removed joint joint_1
- removed joint joint_2
- removed joint joint_3
- removed joint joint_4
- added joint base: type continuous, parent base_link, child link_1, origin xyz=0 0.050345 0 rpy=0 0 3.1416, axis 0 -1 0, limit lower=0 upper=0 effort=0 velocity=0
- added joint elbow: type continuous, parent link_2, child link_3, origin xyz=0.1768 -0.3469 0.259 rpy=-3.1416 -0.69813 3.1416, axis 1 0 0, limit lower=0 upper=0 effort=0 velocity=0
- added joint shoulder: type continuous, parent link_1, child link_2, origin xyz=0.010361 -0.08053 -0.0086937 rpy=0 0 0, axis 0.76604 0 -0.64279, limit lower=0 upper=0 effort=0 velocity=0
- added joint wrist: type continuous, parent link_3, child link_4, origin xyz=-0.031045 0.34673 -0.43413 rpy=-3.1416 0.69813 3.1416, axis -0.76604 0 0.64279, limit lower=0 upper=0 effort=0 velocity=0

Commit message: URDF up to date, grav comp added

File: src/vanderbot/urdf/vanderbot.urdf (robot description, URDF)
Before this commit: robot vanderbot, 6 links, 5 joints
Links:
- added link tip, mass 0.041778; collision mesh filename=package://vanderbot/meshes/link_5.STL; visual mesh filename=package://vanderbot/meshes/link_5.STL
- link base_link: mass None -> 0.80794
- link link_1: mass None -> 0.5361
- link link_2: mass None -> 0.74175
- link link_3: mass None -> 0.44825
- link link_4: mass None -> 0.23876
Joints:
- added joint twist: type continuous, parent link_4, child tip, origin xyz=0 0.07105 -0.04353 rpy=0 0 0, axis 0 -1 0
- joint base: limit lower=0 upper=0 effort=0 velocity=0 -> (none)
- joint elbow: limit lower=0 upper=0 effort=0 velocity=0 -> (none); origin xyz=0.1768 -0.3469 0.259 rpy=-3.1416 -0.69813 3.1416 -> xyz=0.4666 0 0.04505 rpy=0 -1.5708 0
- joint shoulder: axis 0.76604 0 -0.64279 -> 0 0 -1; limit lower=0 upper=0 effort=0 velocity=0 -> (none); origin xyz=0.010361 -0.08053 -0.0086937 rpy=0 0 0 -> xyz=0 -0.08053 -0.013525 rpy=0 0 0
- joint wrist: axis -0.76604 0 0.64279 -> 0 0 -1; limit lower=0 upper=0 effort=0 velocity=0 -> (none); origin xyz=-0.031045 0.34673 -0.43413 rpy=-3.1416 0.69813 3.1416 -> xyz=-0.031045 0 -0.5556 rpy=0 1.5708 0

Commit message: ikin working

File: src/vanderbot/urdf/vanderbot.urdf (robot description, URDF)
Before this commit: robot vanderbot, 7 links, 6 joints
Joints:
- joint fix: origin xyz=0 0 0 rpy=1.5708 0 0 -> xyz=0 0 0 rpy=1.5708 0 -1.5708

Commit message: added gripper to cad, changed urdf with tip at camera

File: src/vanderbot/urdf/vanderbot.urdf (robot description, URDF)
Before this commit: robot vanderbot, 7 links, 6 joints
Links:
- removed link tip
- removed link world
- added link link_5, mass 0.079101; collision mesh filename=package://vanderbot/meshes/link_5.STL; visual mesh filename=package://vanderbot/meshes/link_5.STL
- added link link_6, mass 62.759; collision mesh filename=package://vanderbot/meshes/link_6.STL; visual mesh filename=package://vanderbot/meshes/link_6.STL
Joints:
- removed joint fix
- added joint tip: type fixed, parent link_5, child link_6, origin xyz=0 0.00455 -0.10875 rpy=0 0 0, axis 0 0 0
- joint elbow: origin xyz=0.4666 0 0.04505 rpy=0 -1.5708 0 -> xyz=0.4666 0 0.04505 rpy=3.1416 -1.5708 0
- joint twist: axis 0 -1 0 -> 0 1 0; child tip -> link_5
- joint wrist: axis 0 0 -1 -> 0 0 1

Commit message: URDF changes

File: src/vanderbot/urdf/vanderbot.urdf (robot description, URDF)
Before this commit: robot vanderbot, 7 links, 6 joints
Links:
- removed link link_5
- removed link link_6
- added link cam, mass 62.759
- added link tip, mass 0.079101; collision mesh filename=package://vanderbot/meshes/link_5.STL; visual mesh filename=package://vanderbot/meshes/link_5.STL
- added link world
Joints:
- removed joint tip
- added joint fix: type fixed, parent world, child base_link, origin xyz=0 0 0 rpy=1.5708 0 -1.5708
- added joint tip_to_cam: type fixed, parent tip, child cam, origin xyz=0 0.00455 -0.10875 rpy=-1.5708 3.1416 0, axis 0 0 0
- joint elbow: origin xyz=0.4666 0 0.04505 rpy=3.1416 -1.5708 0 -> xyz=0.4666 0 0.04505 rpy=0 -1.5708 0
- joint twist: child link_5 -> tip
- joint wrist: axis 0 0 1 -> 0 0 -1

Commit message: Arm Cam Demo

File: src/vanderbot/urdf/vanderbot.urdf (robot description, URDF)
Before this commit: robot vanderbot, 8 links, 7 joints
Links:
- link cam: geometry collision mesh filename=package://vanderbot/meshes/link_6.STL; visual mesh filename=package://vanderbot/meshes/link_6.STL
Joints:
- removed joint tip_to_cam
- added joint tip: type fixed, parent tip, child cam, origin xyz=0 0.00455 -0.10875 rpy=-1.5708 3.1416 0, axis 0 0 0
